File: Hardware/servo.kicad_sch (KiCad schematic)
At the start: 5 parts, among them J3 ServoCH0, J4 ServoCH1

Commit message: cleaned up schematic and bom
Parts:
- D601: renamed from D3; value ~ -> CPDV5_3V3UP_HF
- R601: renamed from R40; value 165R -> 165Ω
- R602: renamed from R41; value 165R -> 165Ω
- renumbered J3 to J601, J4 to J602
Changed lines of the file:
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@@
 (kicad_sch
-	(version 20231120)
+	(version 20250114)
 	(generator "eeschema")
-	(generator_version "8.0")
+	(generator_version "9.0")
 	(paper "A4")
 	(wire
@@
 		(shape input)
 		(at 125.73 81.28 90)
-		(fields_autoplaced yes)
 		(effects
 			(font
@@
 		(shape input)
 		(at 118.11 81.28 90)
-		(fields_autoplaced yes)
 		(effects
 			(font
@@
 		(shape input)
 		(at 152.4 78.74 180)
-		(fields_autoplaced yes)
 		(effects
 			(font
@@
 		(shape input)
 		(at 152.4 93.98 180)
-		(fields_autoplaced yes)
 		(effects
 			(font
@@
 		(dnp no)
 		(fields_autoplaced yes)
-		(property "Reference" "R41"
+		(property "Reference" "R602"
 			(at 158.75 91.44 90)
 			(effects
@@
 			)
 		)
-		(property "Value" "165R"
+		(property "Value" "165Ω"
 			(at 158.75 93.98 90)
 			(effects
@@
 			(project "Chad"
 				(path "/7db990e4-92e1-4f99-b4d2-435bbec1ba83/4bc189a8-fc0b-4b23-bb81-ec8cc2a0e30d"
-					(reference "R41")
+					(reference "R602")
 					(unit 1)
 				)
@@
 		(dnp no)
 		(fields_autoplaced yes)
-		(property "Reference" "D3"
+		(property "Reference" "D601"
 			(at 127.9717 87.2649 0)
 			(effects
@@
 			)
 		)
-		(property "Value" "~"
+		(property "Value" "CPDV5_3V3UP_HF"
 			(at 127.9717 89.17 0)
 			(effects
@@
 			(project "Chad"
 				(path "/7db990e4-92e1-4f99-b4d2-435bbec1ba83/4bc189a8-fc0b-4b23-bb81-ec8cc2a0e30d"
-					(reference "D3")
+					(reference "D601")
 					(unit 2)
 				)
@@
 		(on_board yes)
 		(dnp no)
-		(property "Reference" "#PWR024"
+		(property "Reference" "#PWR0602"
 			(at 125.73 100.33 0)
 			(effects
@@
 			(project "Chad"
 				(path "/7db990e4-92e1-4f99-b4d2-435bbec1ba83/4bc189a8-fc0b-4b23-bb81-ec8cc2a0e30d"
-					(reference "#PWR024")
+					(reference "#PWR0602")
 					(unit 1)
 				)
@@
 		(on_board yes)
 		(dnp no)
-		(property "Reference" "#PWR028"
+		(property "Reference" "#PWR0603"
 			(at 149.86 87.63 0)
 			(effects
@@
 			(project "Chad"
 				(path "/7db990e4-92e1-4f99-b4d2-435bbec1ba83/4bc189a8-fc0b-4b23-bb81-ec8cc2a0e30d"
-					(reference "#PWR028")
+					(reference "#PWR0603")
 					(unit 1)
 				)
@@
 		(on_board yes)
 		(dnp no)
-		(property "Reference" "#PWR087"
+		(property "Reference" "#PWR0606"
 			(at 157.48 101.6 0)
 			(effects
@@
 			(project "Chad"
 				(path "/7db990e4-92e1-4f99-b4d2-435bbec1ba83/4bc189a8-fc0b-4b23-bb81-ec8cc2a0e30d"
-					(reference "#PWR087")
+					(reference "#PWR0606")
 					(unit 1)
 				)
@@
 		(on_board yes)
 		(dnp no)
-		(property "Reference" "#PWR086"
+		(property "Reference" "#PWR0605"
 			(at 157.48 86.36 0)
 			(effects
@@
 			(project "Chad"
 				(path "/7db990e4-92e1-4f99-b4d2-435bbec1ba83/4bc189a8-fc0b-4b23-bb81-ec8cc2a0e30d"
-					(reference "#PWR086")
+					(reference "#PWR0605")
 					(unit 1)
 				)
@@
 		(on_board yes)
 		(dnp no)
-		(property "Reference" "J3"
+		(property "Reference" "J601"
 			(at 166.37 77.47 0)
 			(effects
@@
 			(project "Chad"
 				(path "/7db990e4-92e1-4f99-b4d2-435bbec1ba83/4bc189a8-fc0b-4b23-bb81-ec8cc2a0e30d"
-					(reference "J3")
+					(reference "J601")
 					(unit 1)
 				)
@@
 		(on_board yes)
 		(dnp no)
-		(property "Reference" "J4"
+		(property "Reference" "J602"
 			(at 166.37 92.71 0)
 			(effects
@@
 			(project "Chad"
 				(path "/7db990e4-92e1-4f99-b4d2-435bbec1ba83/4bc189a8-fc0b-4b23-bb81-ec8cc2a0e30d"
-					(reference "J4")
+					(reference "J602")
 					(unit 1)
 				)
@@
 		(on_board yes)
 		(dnp no)
-		(property "Reference" "D3"
+		(property "Reference" "D601"
 			(at 116.078 87.63 0)
 			(effects
@@
 			)
 		)
-		(property "Value" "~"
+		(property "Value" "CPDV5_3V3UP_HF"
 			(at 115.57 88.9 0)
 			(effects
@@
 			(project "Chad"
 				(path "/7db990e4-92e1-4f99-b4d2-435bbec1ba83/4bc189a8-fc0b-4b23-bb81-ec8cc2a0e30d"
-					(reference "D3")
+					(reference "D601")
 					(unit 1)
 				)
@@
 		(on_board yes)
 		(dnp no)
-		(property "Reference" "R40"
+		(property "Reference" "R601"
 			(at 158.496 76.454 90)
 			(effects
@@
 			)
 		)
-		(property "Value" "165R"
+		(property "Value" "165Ω"
 			(at 158.496 78.994 90)
 			(effects
@@
 			(project "Chad"
 				(path "/7db990e4-92e1-4f99-b4d2-435bbec1ba83/4bc189a8-fc0b-4b23-bb81-ec8cc2a0e30d"
-					(reference "R40")
+					(reference "R601")
 					(unit 1)
 				)
@@
 		(on_board yes)
 		(dnp no)
-		(property "Reference" "#PWR023"
+		(property "Reference" "#PWR0601"
 			(at 118.11 100.33 0)
 			(effects
@@
 			(project "Chad"
 				(path "/7db990e4-92e1-4f99-b4d2-435bbec1ba83/4bc189a8-fc0b-4b23-bb81-ec8cc2a0e30d"
-					(reference "#PWR023")
+					(reference "#PWR0601")
 					(unit 1)
 				)
@@
 		(on_board yes)
 		(dnp no)
-		(property "Reference" "#PWR029"
+		(property "Reference" "#PWR0604"
 			(at 152.4 102.87 0)
 			(effects
@@
 			(project "Chad"
 				(path "/7db990e4-92e1-4f99-b4d2-435bbec1ba83/4bc189a8-fc0b-4b23-bb81-ec8cc2a0e30d"
-					(reference "#PWR029")
-					(unit 1)
-				)
+					(reference "#PWR0604")
+					(unit 1)
+				)

Commit message: continued
Parts:
- D601: value CPDV5_3V3UP_HF -> CPDV5-3V3UP-HF
Changed lines of the file:
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@@
 			)
 		)
-		(property "Value" "CPDV5_3V3UP_HF"
+		(property "Value" "CPDV5-3V3UP-HF"
 			(at 127.9717 89.17 0)
 			(effects
@@
 			)
 		)
-		(property "Value" "CPDV5_3V3UP_HF"
+		(property "Value" "CPDV5-3V3UP-HF"
 			(at 115.57 88.9 0)
 			(effects
